Commit message: Split workstation launch files and added UR5e workstation.

File: coro_descriptions/urdf/common/2f_coupling.urdf.xacro (robot description, xacro)
@@ -38,5 +38,5 @@
 	        <!-- Mount the gripper to the coupling -->
 	        <link name="${prefix}coupling_gripper_fix"/>
-	        <joint name="coupling_to_fts" type="fixed">
+	        <joint name="coupling_to_gripper" type="fixed">
 	        	<parent link="${prefix}2f_coupling"/>
 	        	<child link="${prefix}coupling_gripper_fix"/>

File: coro_descriptions/urdf/workstations/ur5_workstation.urdf.xacro (robot description, xacro)
@@ -12,6 +12,5 @@
 	</joint>
 	<!-- ROBOT -->
-	<!--<xacro:arg name="kinematics_config" default="$(find ur5_2f85_moveit_config)/../descriptions/ur5/ur5_calibration.yaml"/>
-	<xacro:include filename="$(find ur_e_description)/urdf/ur5e.urdf.xacro" kinematics_file="${load_yaml('$(arg kinematics_config)')}"/>-->
+	<xacro:arg name="kinematics_config" default="$(find ur_description)/config/ur5_default.yaml"/>
 	<xacro:include filename="$(find ur_description)/urdf/ur5.urdf.xacro"/>
 	<xacro:ur5_robot prefix="" joint_limited="true"
@@ -22,5 +21,6 @@
     		wrist_2_lower_limit="${-pi}" wrist_2_upper_limit="${pi}"
     		wrist_3_lower_limit="${-pi}" wrist_3_upper_limit="${pi}"
-    		transmission_hw_interface="hardware_interface/PositionJointInterface"/>
+    		transmission_hw_interface="hardware_interface/PositionJointInterface"
+    		kinematics_file="${load_yaml('$(arg kinematics_config)')}"/>
 	<joint name="robot_to_table" type="fixed">
 		<parent link="middle_robot_mount"/>
