Commit message: Got the hw and sim ur5 working. Still missing hw gripper.

File: coro_descriptions/urdf/common/coro_3arms_table.urdf.xacro (robot description, xacro)
@@ -6,5 +6,6 @@
 		</material>
 	        <!-- Base -->
-		<link name="${prefix}table_base">
+	        <link name="${prefix}table_base"/>
+		<link name="${prefix}table_base_link">
 			<visual>
 				<origin xyz="0 0 ${0.159/2}" rpy="0 0 0"/>
@@ -31,4 +32,9 @@
     			<material>Gazebo/Grey</material>
   		</gazebo>
+  		<joint name="table_root" type="fixed">
+	        	<parent link="${prefix}table_base"/>
+	        	<child link="${prefix}table_base_link"/>
+	        	<origin xyz="0 0 0" rpy="0 0 0"/>
+        	</joint>
 	        <!-- Workspace column -->
 		<link name="${prefix}workspace_column">
@@ -58,5 +64,5 @@
   		</gazebo>
 	        <joint name="workspace_column_to_base" type="fixed">
-	        	<parent link="${prefix}table_base"/>
+	        	<parent link="${prefix}table_base_link"/>
 	        	<child link="${prefix}workspace_column"/>
 	        	<origin xyz="0 0.245 0.159" rpy="0 0 0"/>
@@ -151,5 +157,5 @@
   		</gazebo>
 	        <joint name="robot_column_to_base" type="fixed">
-	        	<parent link="${prefix}table_base"/>
+	        	<parent link="${prefix}table_base_link"/>
 	        	<child link="${prefix}robot_column"/>
 	        	<origin xyz="0 -0.251 0.159" rpy="0 0 0"/>

File: coro_descriptions/urdf/workstations/ur5_workstation.urdf.xacro (robot description, xacro)
@@ -51,7 +51,7 @@
     	<link name="tcp"/>
     	<joint name="tcp_to_gripper" type="fixed">
-    		<parent link="gripper_base_link"/>
+    		<parent link="tool0"/>
     		<child link="tcp"/>
-    		<origin xyz="0 0 0.15" rpy="0 0 0"/>
+    		<origin xyz="0 0 0.19" rpy="0 0 0"/>
 	</joint>
 	<!-- GAZEBO -->
