Commit message: Added ur5e_sim_workstation

File: coro_descriptions/urdf/common/coro_small_vention_table.urdf.xacro (robot description, xacro)
@@ -3,29 +3,29 @@
 	<xacro:macro name="coro_small_vention_table" params="prefix">
 	        <!-- Table -->
-		<link name="${prefix}table">
+		<link name="${prefix}table_base">
 			<visual>
 				<origin xyz="0 0 0.001" rpy="0 0 0"/> <!-- The Z-plane of the table is slightly too high. -->
 				<geometry>
-	                    		<mesh filename="package://coro_descriptions/meshes/small_vention_table.dae"/>
-	                	</geometry>
+					<mesh filename="package://coro_descriptions/meshes/small_vention_table.dae"/>
+				</geometry>
 			</visual>
 			<collision>
-	                	<origin xyz="0 0 0.001" rpy="0 0 0"/> <!-- The Z-plane of the table is slightly too high. -->
+				<origin xyz="0 0 0.001" rpy="0 0 0"/> <!-- The Z-plane of the table is slightly too high. -->
 				<geometry>
-	                    		<mesh filename="package://coro_descriptions/meshes/small_vention_table.dae"/>
-	                	</geometry>
-	            	</collision>
-	            	<inertial>
-	                	<origin xyz="0 0 0" rpy="0 0 0"/>
-	                	<mass value="20"/>
-	                	<inertia ixx="1" ixy="0" ixz="0"
-	                	  	 iyx="0" iyy="1" iyz="0"
-	                	  	 izx="0" izy="0" izz="1"/>
-	            	</inertial>
+					<mesh filename="package://coro_descriptions/meshes/small_vention_table.dae"/>
+				</geometry>
+			</collision>
+			<inertial>
+				<origin xyz="0 0 0" rpy="0 0 0"/>
+				<mass value="20"/>
+				<inertia ixx="1" ixy="0" ixz="0"
+					iyx="0" iyy="1" iyz="0"
+					izx="0" izy="0" izz="1"/>
+				</inertial>
 	        </link>
 	        <!-- Robot mount -->
 	        <link name="${prefix}robot_mount"/>
 	        <joint name="robot_mount" type="fixed">
-	        	<parent link="${prefix}table"/>
+	        	<parent link="${prefix}table_base"/>
 	        	<child link="${prefix}robot_mount"/>
 	        	<origin xyz="-0.3375 0 0.99234" rpy="0 0 0"/>  <!-- The Z-plane of the table is slightly too high. The true Z-origin is 0.099134. -->

File: coro_descriptions/urdf/workstations/ur5e_workstation.urdf.xacro (robot description, xacro)
@@ -21,10 +21,10 @@
 	<xacro:include filename="$(find coro_descriptions)/urdf/common/2f_coupling.urdf.xacro"/>
 	<xacro:coupling_robotiq_2f prefix="" parent="tool0">
-		<origin xyz="0 0 -0.0045" rpy="0 0 0"/>
+		<origin xyz="0 0 0.0045" rpy="0 0 1.5708"/>
 	</xacro:coupling_robotiq_2f>
 	<!-- GRIPPER -->
 	<xacro:include filename="$(find robotiq_85_description)/urdf/robotiq_85_gripper.urdf.xacro"/>
 	<xacro:robotiq_85_gripper prefix="" parent="coupling_gripper_fix">
-		<origin xyz="0 0 0" rpy="0 1.5708 0"/>
+		<origin xyz="0 0 0.0108" rpy="0 -1.5708 0"/>
 	</xacro:robotiq_85_gripper>
 	<link name="tcp"/>

Commit message: Updated small_vention_table mesh

File: coro_descriptions/urdf/common/coro_small_vention_table.urdf.xacro (robot description, xacro)
@@ -5,5 +5,5 @@
 		<link name="${prefix}table_base">
 			<visual>
-				<origin xyz="0 0 0.001" rpy="0 0 0"/> <!-- The Z-plane of the table is slightly too high. -->
+				<origin xyz="0 0 0" rpy="0 0 0"/>
 				<geometry>
 					<mesh filename="package://coro_descriptions/meshes/small_vention_table.dae"/>
@@ -11,5 +11,5 @@
 			</visual>
 			<collision>
-				<origin xyz="0 0 0.001" rpy="0 0 0"/> <!-- The Z-plane of the table is slightly too high. -->
+				<origin xyz="0 0 0" rpy="0 0 0"/>
 				<geometry>
 					<mesh filename="package://coro_descriptions/meshes/small_vention_table.dae"/>
@@ -29,5 +29,5 @@
 	        	<parent link="${prefix}table_base"/>
 	        	<child link="${prefix}robot_mount"/>
-	        	<origin xyz="-0.3375 0 0.99234" rpy="0 0 0"/>  <!-- The Z-plane of the table is slightly too high. The true Z-origin is 0.099134. -->
+				<origin xyz="-0.0093 0.3375 0.99275" rpy="0 0 3.1416"/>  <!-- Coordinates taken from a CAD assembly -->
         	</joint>
 	</xacro:macro>
