Commit message: Added ur10_workstation image and cleaned up old ur5e_workstation files

File: coro_descriptions/urdf/workstations/ur5e_workstation.urdf.xacro (robot description, xacro)
@@ -1,4 +1,4 @@
 <?xml version="1.0" ?>
-<robot name="ur5e_2f85" xmlns:xacro="http://ros.org/wiki/xacro">
+<robot name="ur5_2f85" xmlns:xacro="http://ros.org/wiki/xacro">
 	<!-- WORLD -->
 	<link name="world"/>
@@ -8,19 +8,9 @@
 	<joint name="table_to_world" type="fixed">
 		<parent link="world"/>
-		<child link="table"/>
+		<child link="table_base"/>
 		<origin xyz="0 0 0" rpy="0 0 0"/>
 	</joint>
 	<!-- ROBOT -->
-	<xacro:arg name="kinematics_config" default="$(find ur_e_description)/config/ur5e_default.yaml"/>
-	<xacro:include filename="$(find ur_e_description)/urdf/ur5e.urdf.xacro"/>
-	<xacro:ur5e_robot prefix="" joint_limited="true"
-    		shoulder_pan_lower_limit="${-pi}" shoulder_pan_upper_limit="${pi}"
-    		shoulder_lift_lower_limit="${-pi}" shoulder_lift_upper_limit="${pi}"
-    		elbow_joint_lower_limit="${-pi}" elbow_joint_upper_limit="${pi}"
-    		wrist_1_lower_limit="${-pi}" wrist_1_upper_limit="${pi}"
-    		wrist_2_lower_limit="${-pi}" wrist_2_upper_limit="${pi}"
-    		wrist_3_lower_limit="${-pi}" wrist_3_upper_limit="${pi}"
-    		transmission_hw_interface="hardware_interface/PositionJointInterface"
-    		kinematics_file="${load_yaml('$(arg kinematics_config)')}"/>
+	<xacro:include filename="$(find ur_description)/urdf/ur5e.xacro"/>
 	<joint name="robot_to_table" type="fixed">
 		<parent link="robot_mount"/>
@@ -31,16 +21,16 @@
 	<xacro:include filename="$(find coro_descriptions)/urdf/common/2f_coupling.urdf.xacro"/>
 	<xacro:coupling_robotiq_2f prefix="" parent="tool0">
-		<origin xyz="0 0 0.0075" rpy="3.1416 0 0"/>
-    	</xacro:coupling_robotiq_2f>
+		<origin xyz="0 0 -0.0045" rpy="0 0 0"/>
+	</xacro:coupling_robotiq_2f>
 	<!-- GRIPPER -->
 	<xacro:include filename="$(find robotiq_85_description)/urdf/robotiq_85_gripper.urdf.xacro"/>
 	<xacro:robotiq_85_gripper prefix="" parent="coupling_gripper_fix">
-		<origin xyz="0 0 0" rpy="0 1.5708 1.5708"/>
-    	</xacro:robotiq_85_gripper>
-    	<link name="tcp"/>
-    	<joint name="tcp_to_gripper" type="fixed">
-    		<parent link="gripper_base_link"/>
-    		<child link="tcp"/>
-    		<origin xyz="0 0 0.15" rpy="0 0 0"/>
+		<origin xyz="0 0 0" rpy="0 1.5708 0"/>
+	</xacro:robotiq_85_gripper>
+	<link name="tcp"/>
+	<joint name="tcp_to_gripper" type="fixed">
+		<parent link="tool0"/>
+		<child link="tcp"/>
+		<origin xyz="0 0 0.165" rpy="0 0 0"/>
 	</joint>
 	<!-- GAZEBO -->
